File: Power & Misc.sch (KiCad schematic (older format))
At the start: 40 parts

Commit message: Motor capacitors, test points, jumpers
Parts:
- removed C?: 100n, Resistors_SMD:R_0603, symbol Device:C
- removed C?: 1u, Resistors_SMD:R_0603, symbol Device:C
- removed C?: 300pf, Resistors_SMD:R_0805, symbol Device:C
- removed R?: 10k, symbol Device:R
- removed R? (x2): 1k, symbol Device:R
- removed R? (x2): 220, symbol Device:R
- removed R?: 1k, Resistors_SMD:R_0805, symbol Device:R
- removed TP?: TEST, symbol ec_2b_rescue:TEST
- removed U?: MCP1501, symbol ec_2b_rescue:MCP1501
- gave numbers to parts that had none: 17
Connections:
- net +12V: now also D?.2 (A)
- net +3V3: now also D?.2 (A)
- net led0: now also D?.2 (A)
- net led1: now also D?.2 (A)
Other:
- note removed: "3v3 Reference"
- moved on the sheet: TP?
